File: example/complex.kicad_pcb (KiCad board)
At the start: 4 copper layers, 100 x 80 mm, 165 parts, among them J1 Conn_01x02, J2 Conn_01x02, J3 USB_B_Mini, J4 Conn_01x02, J5 Conn_01x02, J6 Conn_01x03, J8 Conn_01x14, J9 Micro_SD_Card, Q1 MMBT3904, Q2 MMBT3904, Q3 MMBT3904, Q4 DMG2301L, Q5 MMBT3904, Q6 MMBT3904, SW1 SW_SPDT, SW2 -, SW3 SW_Push, SW4 Rotary_Encoder_Switch, U1 LM2902, U10 CP2104, U11 ESP32-WROOM-32D, U2 MCP3004, U3 ILX555K, U4 MCP73831-2-OT, U5 TPS55340RTE, U6 TPS55340RTE, U7 AP2115M, U8 MAX809, U9 74LVC2G86

Commit message: Improved docs
Parts:
- removed C10, C11, C12, C13, C14, C15, C16, C17, C18, C19, C20, C21, C8, C9: C, Capacitor_SMD:C_0603_1608Metric
- removed F2: Fuse, Fuse:Fuse_0603_1608Metric
- removed H1, H2, H4, H5, H6, H7, H8: MountingHole, MountingHole:MountingHole_3.2mm_M3_Pad
- removed H3: MountingHole, infin1d:logo
- removed J1, J4, J5: Conn_01x02, Connector_PinHeader_2.54mm:PinHeader_1x02_P2.54mm_Vertical
- removed J2: Conn_01x02, Connector_JST:JST_PH_S2B-PH-K_1x02_P2.00mm_Horizontal
- removed J3: USB_B_Mini, Connector_USB:USB_Mini-B_Wuerth_65100516121_Horizontal
- removed J6: Conn_01x03, Connector_PinHeader_2.54mm:PinHeader_1x03_P2.54mm_Vertical
- removed J8: Conn_01x14, infin1d:ILI9341-2_8
- removed J9: Micro_SD_Card, GH4:GCT-MEM2055-00-190-01-A
- removed L1, L2: L, Inductor_SMD:L_1206_3216Metric
- removed Q1, Q2, Q3, Q5, Q6: MMBT3904, Package_TO_SOT_SMD:SOT-23
- removed Q4: DMG2301L, Package_TO_SOT_SMD:SOT-23
- removed R10, R11, R12, R13, R14, R15, R17, R18, R19, R20, R21, R22, R23, R24, R25, R26, R8, R9: 100, Resistor_SMD:R_0603_1608Metric
- removed R16, R36, R38, R71, R74: 0, Resistor_SMD:R_0603_1608Metric
- removed R27, R28, R29, R30, R31, R32, R33, R34, R35, R37, R39, R40, R41, R42, R43, R44, R45, R46, R47, R48, R49, R50, R51, R52, R53, R54, R55, R56, R57, R58, R59, R60, R62, R63, R64, R65, R66, R67, R68, R69, R70, R76, R77, R78, R79, R80: R_US, Resistor_SMD:R_0603_1608Metric
- removed R61, R7, R72, R73, R75: DNP, Resistor_SMD:R_0603_1608Metric
- removed SW2: -, Button_Switch_THT:SW_Tactile_SKHH_Angled
- removed SW3: SW_Push, Button_Switch_SMD:SW_Push_1P1T_NO_6x6mm_H9.5mm
- removed SW4: Rotary_Encoder_Switch, GH1:PEC11R
- removed TP1, TP10, TP11, TP2, TP3, TP4, TP5, TP6, TP7, TP8, TP9: TestPoint, TestPoint:TestPoint_Pad_D1.0mm
- removed U10: CP2104, Package_DFN_QFN:QFN-24-1EP_4x4mm_P0.5mm_EP2.6x2.6mm
- removed U11: ESP32-WROOM-32D, RF_Module:ESP32-WROOM-32
- removed U2: MCP3004, Package_SO:TSSOP-14_4.4x5mm_P0.65mm
- removed U3: ILX555K, Package_DIP:DIP-22_W10.16mm
- removed U4: MCP73831-2-OT, Package_TO_SOT_SMD:SOT-23-5
- removed U5, U6: TPS55340RTE, Package_DFN_QFN:WQFN-16-1EP_3x3mm_P0.5mm_EP1.75x1.75mm_ThermalVias
- removed U7: AP2115M, Package_SO:SOIC-8_3.9x4.9mm_P1.27mm
- removed U8: MAX809, Package_TO_SOT_SMD:SOT-23
- removed U9: 74LVC2G86, Package_SO:TSSOP-8_3x3mm_P0.65mm
- added D13: SOD-123, Diode_SMD:D_SOD-123, B.Cu at (227.0, -93.7)
- added D14: SOD-123, Diode_SMD:D_SOD-123, B.Cu at (246.1, -93.7)
- added D15: SOD-123, Diode_SMD:D_SOD-123, B.Cu at (265.1, -93.7)
- added D16: SOD-123, Diode_SMD:D_SOD-123, B.Cu at (284.2, -93.7)
- added D17: SOD-123, Diode_SMD:D_SOD-123, B.Cu at (287.3, -93.7)
- added D18: SOD-123, Diode_SMD:D_SOD-123, B.Cu at (350.8, -93.6)
- added D19: SOD-123, Diode_SMD:D_SOD-123, B.Cu at (369.9, -93.6)
- added D20: SOD-123, Diode_SMD:D_SOD-123, B.Cu at (388.1, -93.7)
- added D21: SOD-123, Diode_SMD:D_SOD-123, B.Cu at (84.1, -74.6)
- added D22: SOD-123, Diode_SMD:D_SOD-123, B.Cu at (103.2, -74.6)
- added D23: SOD-123, Diode_SMD:D_SOD-123, B.Cu at (122.2, -74.6)
- added D24: SOD-123, Diode_SMD:D_SOD-123, B.Cu at (141.3, -74.6)
- added D25: SOD-123, Diode_SMD:D_SOD-123, B.Cu at (160.3, -74.6)
- added D26: SOD-123, Diode_SMD:D_SOD-123, B.Cu at (179.4, -74.6)
- added D27: SOD-123, Diode_SMD:D_SOD-123, B.Cu at (198.4, -74.6)
- added D28: SOD-123, Diode_SMD:D_SOD-123, B.Cu at (217.5, -74.6)
- added D29: SOD-123, Diode_SMD:D_SOD-123, B.Cu at (236.5, -74.6)
- added D30: SOD-123, Diode_SMD:D_SOD-123, B.Cu at (255.6, -74.6)
- added D31: SOD-123, Diode_SMD:D_SOD-123, B.Cu at (274.6, -74.6)
- added D32: SOD-123, Diode_SMD:D_SOD-123, B.Cu at (293.7, -74.6)
- added D33: SOD-123, Diode_SMD:D_SOD-123, B.Cu at (300.8, -74.6)
- added D34: SOD-123, Diode_SMD:D_SOD-123, B.Cu at (350.8, -74.6)
- added D35: SOD-123, Diode_SMD:D_SOD-123, B.Cu at (369.9, -74.5)
- added D36: SOD-123, Diode_SMD:D_SOD-123, B.Cu at (388.1, -74.6)
- added D37: SOD-123, Diode_SMD:D_SOD-123, B.Cu at (27.0, -55.6)
- added D38: SOD-123, Diode_SMD:D_SOD-123, B.Cu at (62.7, -55.6)
- added D39: SOD-123, Diode_SMD:D_SOD-123, B.Cu at (88.9, -55.6)
- added D40: SOD-123, Diode_SMD:D_SOD-123, B.Cu at (108.0, -55.6)
- added D41: SOD-123, Diode_SMD:D_SOD-123, B.Cu at (127.0, -55.6)
- added D42: SOD-123, Diode_SMD:D_SOD-123, B.Cu at (146.1, -55.6)
- added D43: SOD-123, Diode_SMD:D_SOD-123, B.Cu at (165.1, -55.6)
- added D44: SOD-123, Diode_SMD:D_SOD-123, B.Cu at (184.2, -55.6)
- added D45: SOD-123, Diode_SMD:D_SOD-123, B.Cu at (203.2, -55.6)
- added D46: SOD-123, Diode_SMD:D_SOD-123, B.Cu at (222.2, -55.6)
- added D47: SOD-123, Diode_SMD:D_SOD-123, B.Cu at (241.3, -55.6)
- added D48: SOD-123, Diode_SMD:D_SOD-123, B.Cu at (260.4, -55.6)
- added D49: SOD-123, Diode_SMD:D_SOD-123, B.Cu at (279.4, -55.6)
- added D50: SOD-123, Diode_SMD:D_SOD-123, B.Cu at (311.1, -55.6)
- added D51: SOD-123, Diode_SMD:D_SOD-123, B.Cu at (323.1, -95.2)
- added D52: SOD-123, Diode_SMD:D_SOD-123, B.Cu at (27.0, -36.5)
- added D53: SOD-123, Diode_SMD:D_SOD-123, B.Cu at (42.1, -36.5)
- added D54: SOD-123, Diode_SMD:D_SOD-123, B.Cu at (79.4, -36.5)
- added D55: SOD-123, Diode_SMD:D_SOD-123, B.Cu at (98.4, -36.5)
- added D56: SOD-123, Diode_SMD:D_SOD-123, B.Cu at (117.5, -36.5)
- added D57: SOD-123, Diode_SMD:D_SOD-123, B.Cu at (136.5, -36.5)
- added D58: SOD-123, Diode_SMD:D_SOD-123, B.Cu at (155.6, -36.5)
- added D59: SOD-123, Diode_SMD:D_SOD-123, B.Cu at (174.6, -36.5)
- added D60: SOD-123, Diode_SMD:D_SOD-123, B.Cu at (193.7, -36.5)
- added D61: SOD-123, Diode_SMD:D_SOD-123, B.Cu at (212.7, -36.5)
- added D62: SOD-123, Diode_SMD:D_SOD-123, B.Cu at (231.8, -36.5)
- added D63: SOD-123, Diode_SMD:D_SOD-123, B.Cu at (250.8, -36.5)
- added D64: SOD-123, Diode_SMD:D_SOD-123, B.Cu at (269.9, -36.5)
- added D65: SOD-123, Diode_SMD:D_SOD-123, B.Cu at (305.6, -36.5)
- added D66: SOD-123, Diode_SMD:D_SOD-123, B.Cu at (322.3, -36.5)
- added D67: SOD-123, Diode_SMD:D_SOD-123, B.Cu at (369.9, -36.5)
- added D68: SOD-123, Diode_SMD:D_SOD-123, B.Cu at (27.0, -17.5)
- added D69: SOD-123, Diode_SMD:D_SOD-123, B.Cu at (60.3, -17.5)
- added D70: SOD-123, Diode_SMD:D_SOD-123, B.Cu at (84.1, -17.5)
- added D71: SOD-123, Diode_SMD:D_SOD-123, B.Cu at (108.0, -17.5)
- added D72: SOD-123, Diode_SMD:D_SOD-123, B.Cu at (188.9, -17.5)
- added D73: SOD-123, Diode_SMD:D_SOD-123, B.Cu at (248.4, -17.5)
- added D74: SOD-123, Diode_SMD:D_SOD-123, B.Cu at (272.3, -17.5)
- added D75: SOD-123, Diode_SMD:D_SOD-123, B.Cu at (296.1, -17.4)
- added D76: SOD-123, Diode_SMD:D_SOD-123, B.Cu at (319.9, -17.4)
- added D77: SOD-123, Diode_SMD:D_SOD-123, B.Cu at (350.8, -17.5)
- added D78: SOD-123, Diode_SMD:D_SOD-123, B.Cu at (369.9, -17.5)
- added D79: SOD-123, Diode_SMD:D_SOD-123, B.Cu at (388.1, -17.5)
- added MX1: MX-NoLED, MX_Alps_Hybrid:MX-1U-NoLED, F.Cu at (19.1, -95.2)
- added MX10: MX-NoLED, MX_Alps_Hybrid:MX-1U-NoLED, F.Cu at (200.0, -95.2)
- added MX11: MX-NoLED, MX_Alps_Hybrid:MX-1U-NoLED, F.Cu at (219.1, -95.2)
- added MX12: MX-NoLED, MX_Alps_Hybrid:MX-1U-NoLED, F.Cu at (238.1, -95.2)
- added MX13: MX-NoLED, MX_Alps_Hybrid:MX-1U-NoLED, F.Cu at (257.2, -95.2)
- added MX14: MX-NoLED, MX_Alps_Hybrid:MX-1U-NoLED, F.Cu at (276.2, -95.2)
- added MX15: MX-NoLED, MX_Alps_Hybrid:MX-1U-NoLED, F.Cu at (295.3, -95.2)
- added MX16: MX-NoLED, MX_Alps_Hybrid:MX-2U-NoLED, F.Cu at (304.8, -95.2)
- added MX17: MX-NoLED, MX_Alps_Hybrid:MX-1U-NoLED, F.Cu at (342.9, -95.2)
- added MX18: MX-NoLED, MX_Alps_Hybrid:MX-1U-NoLED, F.Cu at (361.9, -95.2)
- added MX19: MX-NoLED, MX_Alps_Hybrid:MX-1U-NoLED, F.Cu at (381.0, -95.2)
- added MX2: MX-NoLED, MX_Alps_Hybrid:MX-1U-NoLED, F.Cu at (47.6, -95.2)
- added MX20: MX-NoLED, MX_Alps_Hybrid:MX-1U-NoLED, F.Cu at (19.1, -76.2)
- added MX21: MX-NoLED, MX_Alps_Hybrid:MX-1U-NoLED, F.Cu at (52.4, -76.2)
- added MX22: MX-NoLED, MX_Alps_Hybrid:MX-1U-NoLED, F.Cu at (76.2, -76.2)
- added MX23: MX-NoLED, MX_Alps_Hybrid:MX-1U-NoLED, F.Cu at (95.2, -76.2)
- added MX24: MX-NoLED, MX_Alps_Hybrid:MX-1U-NoLED, F.Cu at (114.3, -76.2)
- added MX25: MX-NoLED, MX_Alps_Hybrid:MX-1U-NoLED, F.Cu at (133.3, -76.2)
- added MX26: MX-NoLED, MX_Alps_Hybrid:MX-1U-NoLED, F.Cu at (152.4, -76.2)
- added MX27: MX-NoLED, MX_Alps_Hybrid:MX-1U-NoLED, F.Cu at (171.4, -76.2)
- added MX28: MX-NoLED, MX_Alps_Hybrid:MX-1U-NoLED, F.Cu at (190.5, -76.2)
- added MX29: MX-NoLED, MX_Alps_Hybrid:MX-1U-NoLED, F.Cu at (209.6, -76.2)
- added MX3: MX-NoLED, MX_Alps_Hybrid:MX-1U-NoLED, F.Cu at (66.7, -95.2)
- added MX30: MX-NoLED, MX_Alps_Hybrid:MX-1U-NoLED, F.Cu at (228.6, -76.2)
- added MX31: MX-NoLED, MX_Alps_Hybrid:MX-1U-NoLED, F.Cu at (247.7, -76.2)
- added MX32: MX-NoLED, MX_Alps_Hybrid:MX-1U-NoLED, F.Cu at (266.7, -76.2)
- added MX33: MX-NoLED, MX_Alps_Hybrid:MX-1U-NoLED, F.Cu at (285.8, -76.2)
- added MX34: MX-NoLED, MX_Alps_Hybrid:MX-1U-NoLED, F.Cu at (309.6, -76.2)
- added MX35: MX-NoLED, MX_Alps_Hybrid:MX-ISO, F.Cu at (311.9, -66.7)
- added MX36: MX-NoLED, MX_Alps_Hybrid:MX-1U-NoLED, F.Cu at (342.9, -76.2)
- added MX37: MX-NoLED, MX_Alps_Hybrid:MX-1U-NoLED, F.Cu at (361.9, -76.2)
- added MX38: MX-NoLED, MX_Alps_Hybrid:MX-1U-NoLED, F.Cu at (381.0, -76.2)
- added MX39: MX-NoLED, MX_Alps_Hybrid:MX-1U-NoLED, F.Cu at (19.1, -57.1)
- added MX4: MX-NoLED, MX_Alps_Hybrid:MX-1U-NoLED, F.Cu at (85.7, -95.2)
- added MX40: MX-NoLED, MX_Alps_Hybrid:MX-1U-NoLED, F.Cu at (50.0, -57.1)
- added MX41: MX-NoLED, MX_Alps_Hybrid:MX-1U-NoLED, F.Cu at (54.8, -57.1)
- added MX42: MX-NoLED, MX_Alps_Hybrid:MX-1U-NoLED, F.Cu at (81.0, -57.1)
- added MX43: MX-NoLED, MX_Alps_Hybrid:MX-1U-NoLED, F.Cu at (100.0, -57.1)
- added MX44: MX-NoLED, MX_Alps_Hybrid:MX-1U-NoLED, F.Cu at (119.1, -57.1)
- added MX45: MX-NoLED, MX_Alps_Hybrid:MX-1U-NoLED, F.Cu at (138.1, -57.1)
- added MX46: MX-NoLED, MX_Alps_Hybrid:MX-1U-NoLED, F.Cu at (157.2, -57.1)
- added MX47: MX-NoLED, MX_Alps_Hybrid:MX-1U-NoLED, F.Cu at (176.2, -57.1)
- added MX48: MX-NoLED, MX_Alps_Hybrid:MX-1U-NoLED, F.Cu at (195.3, -57.1)
- added MX49: MX-NoLED, MX_Alps_Hybrid:MX-1U-NoLED, F.Cu at (214.3, -57.1)
- added MX5: MX-NoLED, MX_Alps_Hybrid:MX-1U-NoLED, F.Cu at (104.8, -95.2)
- added MX50: MX-NoLED, MX_Alps_Hybrid:MX-1U-NoLED, F.Cu at (233.4, -57.1)
- added MX51: MX-NoLED, MX_Alps_Hybrid:MX-1U-NoLED, F.Cu at (252.4, -57.1)
- added MX52: MX-NoLED, MX_Alps_Hybrid:MX-1U-NoLED, F.Cu at (271.5, -57.1)
- added MX53: MX-NoLED, MX_Alps_Hybrid:MX-1U-NoLED, F.Cu at (290.5, -57.1)
- added MX54: MX-NoLED, MX_Alps_Hybrid:MX-2U-NoLED, F.Cu at (302.4, -57.1)
- added MX55: MX-NoLED, MX_Alps_Hybrid:MX-1U-NoLED, F.Cu at (314.3, -95.2)
- added MX56: MX-NoLED, MX_Alps_Hybrid:MX-1U-NoLED, F.Cu at (19.1, -38.1)
- added MX57: MX-NoLED, MX_Alps_Hybrid:MX-1U-NoLED, F.Cu at (50.0, -38.1)
- added MX58: MX-NoLED, MX_Alps_Hybrid:MX-2U-NoLED, F.Cu at (59.5, -38.1)
- added MX59: MX-NoLED, MX_Alps_Hybrid:MX-1U-NoLED, F.Cu at (71.4, -38.1)
- added MX6: MX-NoLED, MX_Alps_Hybrid:MX-1U-NoLED, F.Cu at (123.8, -95.2)
- added MX60: MX-NoLED, MX_Alps_Hybrid:MX-1U-NoLED, F.Cu at (90.5, -38.1)
- added MX61: MX-NoLED, MX_Alps_Hybrid:MX-1U-NoLED, F.Cu at (109.5, -38.1)
- added MX62: MX-NoLED, MX_Alps_Hybrid:MX-1U-NoLED, F.Cu at (128.6, -38.1)
- added MX63: MX-NoLED, MX_Alps_Hybrid:MX-1U-NoLED, F.Cu at (147.6, -38.1)
- added MX64: MX-NoLED, MX_Alps_Hybrid:MX-1U-NoLED, F.Cu at (166.7, -38.1)
- added MX65: MX-NoLED, MX_Alps_Hybrid:MX-1U-NoLED, F.Cu at (185.7, -38.1)
- added MX66: MX-NoLED, MX_Alps_Hybrid:MX-1U-NoLED, F.Cu at (204.8, -38.1)
- added MX67: MX-NoLED, MX_Alps_Hybrid:MX-1U-NoLED, F.Cu at (223.8, -38.1)
- added MX68: MX-NoLED, MX_Alps_Hybrid:MX-1U-NoLED, F.Cu at (242.9, -38.1)
- added MX69: MX-NoLED, MX_Alps_Hybrid:MX-1U-NoLED, F.Cu at (261.9, -38.1)
- added MX7: MX-NoLED, MX_Alps_Hybrid:MX-1U-NoLED, F.Cu at (142.9, -95.2)
- added MX70: MX-NoLED, MX_Alps_Hybrid:MX-1U-NoLED, F.Cu at (288.1, -38.1)
- added MX71: MX-NoLED, MX_Alps_Hybrid:MX-2U-NoLED, F.Cu at (297.7, -38.1)
- added MX72: MX-NoLED, MX_Alps_Hybrid:MX-1U-NoLED, F.Cu at (314.3, -38.1)
- added MX73: MX-NoLED, MX_Alps_Hybrid:MX-1U-NoLED, F.Cu at (361.9, -38.1)
- added MX74: MX-NoLED, MX_Alps_Hybrid:MX-1U-NoLED, F.Cu at (19.1, -19.1)
- added MX75: MX-NoLED, MX_Alps_Hybrid:MX-1U-NoLED, F.Cu at (50.0, -19.1)
- added MX76: MX-NoLED, MX_Alps_Hybrid:MX-1U-NoLED, F.Cu at (73.8, -19.1)
- added MX77: MX-NoLED, MX_Alps_Hybrid:MX-1U-NoLED, F.Cu at (97.6, -19.1)
- added MX78: MX-NoLED, MX_Alps_Hybrid:MX-6.25U-ReversedStabilizers-NoLED, F.Cu at (169.1, -19.1)
- added MX79: MX-NoLED, MX_Alps_Hybrid:MX-1U-NoLED, F.Cu at (240.5, -19.1)
- added MX8: MX-NoLED, MX_Alps_Hybrid:MX-1U-NoLED, F.Cu at (161.9, -95.2)
- added MX80: MX-NoLED, MX_Alps_Hybrid:MX-1U-NoLED, F.Cu at (264.3, -19.1)
- added MX81: MX-NoLED, MX_Alps_Hybrid:MX-1U-NoLED, F.Cu at (288.1, -19.1)
- added MX82: MX-NoLED, MX_Alps_Hybrid:MX-1U-NoLED, F.Cu at (311.9, -19.1)
- added MX83: MX-NoLED, MX_Alps_Hybrid:MX-1U-NoLED, F.Cu at (342.9, -19.1)
- added MX84: MX-NoLED, MX_Alps_Hybrid:MX-1U-NoLED, F.Cu at (361.9, -19.1)
- added MX85: MX-NoLED, MX_Alps_Hybrid:MX-1U-NoLED, F.Cu at (381.0, -19.1)
- added MX86: MX-NoLED, MX_Alps_Hybrid:MX-1U-NoLED, F.Cu at (52.4, -19.1)
- added MX87: MX-NoLED, MX_Alps_Hybrid:MX-1U-NoLED, F.Cu at (76.2, -19.1)
- added MX88: MX-NoLED, MX_Alps_Hybrid:MX-1U-NoLED, F.Cu at (100.0, -19.1)
- added MX89: MX-NoLED, MX_Alps_Hybrid:MX-7U-ReversedStabilizers-NoLED, F.Cu at (181.0, -19.1)
- added MX9: MX-NoLED, MX_Alps_Hybrid:MX-1U-NoLED, F.Cu at (181.0, -95.2)
- added MX90: MX-NoLED, MX_Alps_Hybrid:MX-1U-NoLED, F.Cu at (261.9, -19.1)
- added MX91: MX-NoLED, MX_Alps_Hybrid:MX-1U-NoLED, F.Cu at (285.8, -19.1)
- added MX92: MX-NoLED, MX_Alps_Hybrid:MX-1U-NoLED, F.Cu at (309.6, -19.1)
- added USB1: HRO-TYPE-C-31-M-12, Type-C:HRO-TYPE-C-31-M-12, B.Cu at (200.0, -112.2)
- added Y1: 16MHz, Crystal:Crystal_SMD_3225-4Pin_3.2x2.5mm, B.Cu at (144.5, -32.6)
- C1, C2: value C -> 22pF; footprint Capacitor_SMD:C_0603_1608Metric -> Capacitor_SMD:C_0805_2012Metric; moved to B.Cu
- C3: value C -> 1uF; footprint Capacitor_SMD:C_0603_1608Metric -> Capacitor_SMD:C_0805_2012Metric; moved to B.Cu
- C4, C5, C6: value C -> 0.1uF; footprint Capacitor_SMD:C_0603_1608Metric -> Capacitor_SMD:C_0805_2012Metric; moved to B.Cu
- C7: value C -> 10uF; footprint Capacitor_SMD:C_0603_1608Metric -> Capacitor_SMD:C_0805_2012Metric; moved to B.Cu
- D1, D2, D3, D4, D5, D6, D7, D8, D9: value D_Schottky -> SOD-123; moved to B.Cu
- D10, D11, D12: value LED -> SOD-123; footprint LED_SMD:LED_0603_1608Metric -> Diode_SMD:D_SOD-123; moved to B.Cu
- F1: value Fuse -> 500mA; footprint Fuse:Fuse_0603_1608Metric -> Fuse:Fuse_1206_3216Metric; moved to B.Cu
- R1, R2: value 100 -> 5.1k; footprint Resistor_SMD:R_0603_1608Metric -> Resistor_SMD:R_0805_2012Metric; moved to B.Cu
- R3: value 100 -> 10k; footprint Resistor_SMD:R_0603_1608Metric -> Resistor_SMD:R_0805_2012Metric; moved to B.Cu
- R4, R5: value 100 -> 22; footprint Resistor_SMD:R_0603_1608Metric -> Resistor_SMD:R_0805_2012Metric; moved to B.Cu
- R6: value 0 -> 10k; footprint Resistor_SMD:R_0603_1608Metric -> Resistor_SMD:R_0805_2012Metric; moved to B.Cu
- SW1: value SW_SPDT -> SW_Push; footprint infin1d:SIP-3 -> random-keyboard-parts:SKQG-1155865; moved to B.Cu
- U1: value LM2902 -> ATmega32U4-AU; footprint Package_SO:TSSOP-14_4.4x5mm_P0.65mm -> Package_QFP:TQFP-44_10x10mm_P0.8mm; moved to B.Cu
- moved D1 228.0 mm to (27.0, -93.7), turned to 90 degrees
- moved F1 227.3 mm to (188.9, -99.1), turned to 90 degrees
- moved D2 219.4 mm to (55.6, -93.7), turned to 90 degrees
- moved R5 213.6 mm to (208.0, -100.6), turned to 270 degrees
- moved D8 212.9 mm to (131.8, -93.7), turned to 90 degrees
- moved D10 209.5 mm to (169.9, -93.7), turned to 90 degrees
- moved D5 208.1 mm to (74.6, -93.7), turned to 90 degrees
- moved R4 205.8 mm to (211.2, -100.6), turned to 90 degrees
- moved D3 202.8 mm to (27.0, -74.6), turned to 90 degrees
- moved D11 197.7 mm to (188.9, -93.7), turned to 90 degrees
- moved D7 192.4 mm to (112.7, -93.7)
- moved D6 189.9 mm to (93.7, -93.7), turned to 90 degrees
- moved D12 187.6 mm to (208.0, -93.7), turned to 90 degrees
- moved D4 184.7 mm to (60.3, -74.6), turned to 90 degrees
- moved D9 174.0 mm to (150.8, -93.7), turned to 90 degrees
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Connections:
- C1 pad 1: VBUS -> Net-(C1-Pad1)
- C2 pad 1: VBUS -> GND
- C2 pad 2: GND -> Net-(C2-Pad2)
- C3 pad 1: Net-(C3-Pad1) -> GND
- C3 pad 2: GND -> Net-(C3-Pad2)
- C4 pad 1: Net-(C4-Pad1) -> +5V
- C5 pad 1: Net-(C5-Pad1) -> +5V
- C6 pad 1: Net-(C6-Pad1) -> +5V
- C7 pad 1: Net-(C7-Pad1) -> +5V
- D1 pad 1: Net-(D1-Pad1) -> ROW0
- D1 pad 2: +5V -> Net-(D1-Pad2)
- D10 pad 1: GND -> ROW0
- D11 pad 1: GND -> ROW0
- D12 pad 1: GND -> ROW0
- D2 pad 1: Net-(D2-Pad1) -> ROW0
- D2 pad 2: +5V -> Net-(D2-Pad2)
- D3 pad 1: Net-(D3-Pad1) -> ROW1
- D3 pad 2: +5V -> Net-(D3-Pad2)
- D4 pad 1: Net-(D4-Pad1) -> ROW1
- D4 pad 2: +5V -> Net-(D4-Pad2)
- D5 pad 1: Net-(D5-Pad1) -> ROW0
- D5 pad 2: +5V -> Net-(D5-Pad2)
- D6 pad 1: Net-(D6-Pad1) -> ROW0
- D6 pad 2: +5V -> Net-(D6-Pad2)
- D7 pad 1: VIN -> ROW0
- D7 pad 2: VBUS -> Net-(D7-Pad2)
- D8 pad 1: Net-(D8-Pad1) -> ROW0
- D9 pad 1: Net-(D9-Pad1) -> ROW0
- F1 pad 1: +BATT -> +5V
- F1 pad 2: Net-(F1-Pad2) -> VCC
- R1 pad 1: Net-(R1-Pad1) -> GND
- R2 pad 1: Net-(R2-Pad1) -> GND
- R2 pad 2: +5V -> Net-(R2-Pad2)
- R3 pad 1: Net-(R2-Pad1) -> +5V
- R3 pad 2: +12V -> Net-(R3-Pad2)
- R4 pad 1: Net-(R1-Pad2) -> Net-(R4-Pad1)
- R4 pad 2: /p3-sensor/VOUT-R -> D+
- R5 pad 1: Net-(R5-Pad1) -> D-
- R5 pad 2: Net-(R1-Pad1) -> Net-(R5-Pad2)
- R6 pad 1: Net-(R6-Pad1) -> GND
- R6 pad 2: +3V3 -> Net-(R6-Pad2)
- SW1 pad 1: Net-(SW1-Pad1) -> GND
- SW1 pad 2: /p1-power/PWR_EN -> Net-(R3-Pad2)
- SW1 pad 3: Net-(SW1-Pad3) -> (no net)
- U1 pad 10: GND -> ROW1
- U1 pad 11: GND -> ROW0
- U1 pad 12: GND -> COL10
- U1 pad 13: Net-(R11-Pad2) -> Net-(R3-Pad2)
- U1 pad 14: Net-(R11-Pad1) -> +5V
- U1 pad 2: Net-(R8-Pad2) -> +5V
- U1 pad 3: GND -> Net-(R5-Pad2)
- U1 pad 4: Net-(R2-Pad1) -> Net-(R4-Pad1)
- U1 pad 6: GND -> Net-(C3-Pad2)
- U1 pad 7: Net-(U1-Pad7) -> +5V
- U1 pad 8: Net-(R1-Pad1) -> Net-(U1-Pad8)
- U1 pad 9: Net-(R1-Pad2) -> ROW2
Routing:
- net ROW0: track 0.00 -> 546.0 mm, vias 0 -> 2
- net ROW4: track 0.00 -> 527.6 mm
- net ROW1: track 0.00 -> 523.4 mm, vias 0 -> 2
- net ROW2: track 0.00 -> 475.6 mm, vias 0 -> 4
- net ROW3: track 0.00 -> 472.9 mm
- net COL1: track 0.00 -> 379.0 mm, vias 0 -> 2
- net COL14: track 0.00 -> 347.8 mm, vias 0 -> 2
- net COL2: track 0.00 -> 340.4 mm, vias 0 -> 2
- net COL16: track 0.00 -> 331.8 mm, vias 0 -> 3
- net COL3: track 0.00 -> 319.0 mm, vias 0 -> 2
- net COL17: track 0.00 -> 315.2 mm, vias 0 -> 2
- net COL15: track 0.00 -> 312.3 mm, vias 0 -> 3
- net COL13: track 0.00 -> 290.8 mm, vias 0 -> 2
- net COL12: track 0.00 -> 260.7 mm, vias 0 -> 2
- net COL0: track 0.00 -> 230.4 mm
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- added copper zone on B.Cu, net GND
- removed copper zone on B.Cu, net (none)
- removed copper zone on In2.Cu, net +12V
- removed copper zone on F.Cu, net +3V3
- removed copper zone on In2.Cu, net +3V3
- removed copper zone on F.Cu, net +5V
- removed copper zone on In2.Cu, net +5V
- removed copper zone on In2.Cu, net +BATT
- removed copper zone on F.Cu, net GND
- removed copper zone on In1.Cu, net GND
- removed copper zone on F.Cu, net Net-(D8-Pad2)
- removed copper zone on F.Cu, net Net-(D9-Pad2)
- removed copper zone on In2.Cu, net VBUS
- removed copper zone on In2.Cu, net VIN
Other:
- board size 100 x 80 mm -> 380 x 100.6 mm
- copper layers 4 -> 2
- net class Default: clearance 0.1524 -> 0.2; trace_width 0.1524 -> 0.25; via_dia 0.6 -> 0.8; via_drill 0.3 -> 0.4
- rule pad_to_mask_clearance: 0.0508 -> 0.051
- rule trace_clearance: 0.1524 -> 0.2
- rule trace_min: 0.1524 -> 0.15
- rule via_min_size: 0.6 -> 0.4
- board text removed: "Infin1D"
- board text removed: "Jarrett Rainier"
- board text removed: "R1 Apr '20"
- board text removed: "jrainimo.com"
